Commit message: initial test on real robot with front 2 wheels

File: description/ros2_control.xacro (robot description, xacro)
@@ -32,5 +32,33 @@
     </xacro:unless> -->
     <!-- <xacro:if value="$(arg sim_mode)"> -->
-    <ros2_control name="GazeboSystem" type="system">
+    <ros2_control name="RealRobot" type="system">
+        <hardware>
+            <plugin>diffdrive_arduino/DiffDriveArduino</plugin>
+            <param name="left_wheel_name">wheel_FL_joint</param>
+            <param name="right_wheel_name">wheel_FR_joint</param>
+            <param name="loop_rate">30</param>
+            <param name="device">/dev/ttyACM0</param>
+            <param name="baud_rate">57600</param>
+            <param name="timeout">1000</param>
+            <param name="enc_counts_per_rev">220</param>
+        </hardware>
+        <joint name="wheel_FL_joint">
+            <command_interface name="velocity">
+                <param name="min">-10</param>
+                <param name="max">10</param>
+            </command_interface>
+            <state_interface name="velocity"/>
+            <state_interface name="position"/>
+        </joint>
+        <joint name="wheel_FR_joint">
+            <command_interface name="velocity">
+                <param name="min">-10</param>
+                <param name="max">10</param>
+            </command_interface>
+            <state_interface name="velocity"/>
+            <state_interface name="position"/>
+        </joint>
+    </ros2_control>
+    <!-- <ros2_control name="GazeboSystem" type="system">
         <hardware>
             <plugin>gazebo_ros2_control/GazeboSystem</plugin>
@@ -68,5 +96,5 @@
             <state_interface name="position"/>
         </joint>
-    </ros2_control>
+    </ros2_control> -->
     <!-- </xacro:if> -->
     <gazebo>

Commit message: working before add simulation switch macro

File: description/ros2_control.xacro (robot description, xacro)
@@ -35,6 +35,8 @@
         <hardware>
             <plugin>diffdrive_arduino/DiffDriveArduino</plugin>
-            <param name="left_wheel_name">wheel_FL_joint</param>
-            <param name="right_wheel_name">wheel_FR_joint</param>
+            <param name="F_left_wheel_name">wheel_FL_joint</param>
+            <param name="F_right_wheel_name">wheel_FR_joint</param>
+            <param name="B_left_wheel_name">wheel_RL_joint</param>
+            <param name="B_right_wheel_name">wheel_RR_joint</param>
             <param name="loop_rate">30</param>
             <param name="device">/dev/ttyACM0</param>
@@ -52,4 +54,20 @@
         </joint>
         <joint name="wheel_FR_joint">
+            <command_interface name="velocity">
+                <param name="min">-10</param>
+                <param name="max">10</param>
+            </command_interface>
+            <state_interface name="velocity"/>
+            <state_interface name="position"/>
+        </joint>
+         <joint name="wheel_RL_joint">
+            <command_interface name="velocity">
+                <param name="min">-10</param>
+                <param name="max">10</param>
+            </command_interface>
+            <state_interface name="velocity"/>
+            <state_interface name="position"/>
+        </joint>
+        <joint name="wheel_RR_joint">
             <command_interface name="velocity">
                 <param name="min">-10</param>
