Commit message: up to video before apply to ros2 control to real robot

File: description/gazebo_control.xacro (robot description, xacro)
@@ -11,4 +11,5 @@
             <wheel_separation>0.22381</wheel_separation>
             <wheel_separation>0.22381</wheel_separation>
+            <!-- dont know if its 0.057 or 0.0625 radius here took 0.057 -->
             <wheel_diameter>0.114</wheel_diameter>
             <wheel_diameter>0.114</wheel_diameter>

File: description/leo.urdf.xacro (robot description, xacro)
@@ -1,6 +1,15 @@
 <?xml version="1.0"?>
 <robot xmlns:xacro="http://www.ros.org/wiki/xacro" name="robot">
-  <xacro:include filename="macros.xacro"/>
-  <xacro:leo/>
-  <xacro:include filename="gazebo_control.xacro" />
+      <!-- <xacro:arg name="use_ros2_control" default="true"/> -->
+      <xacro:include filename="macros.xacro"/>
+      <xacro:leo/>
+      <!-- <xacro:if value="$(arg use_ros2_control)">
+        <xacro:include filename="ros2_control.xacro" />
+      </xacro:if>
+      <xacro:unless value="$(arg use_ros2_control)">
+            <xacro:include filename="gazebo_control.xacro" />
+      </xacro:unless> -->
+      <xacro:include filename="ros2_control.xacro" />
+      <xacro:include filename="lidar.xacro" />
+      <xacro:include filename="camera.xacro" />
 </robot>

File: description/macros.xacro (robot description, xacro)
@@ -1,4 +1,7 @@
 <?xml version="1.0"?>
 <robot xmlns:xacro="http://www.ros.org/wiki/xacro" >
+  <!-- zach, changed all filename to file://$(find my_bot)-->
+  <xacro:include filename="inertial_macros.xacro"/>
+  <!-- zach -->
   <xacro:macro name="leo"
                params="default_antenna:=false
@@ -64,4 +67,12 @@
       </link>
     </xacro:macro>
+    <!-- zach -->
+    <material name="red">
+          <color rgba="1 0 0 1"/>
+    </material>
+    <material name="blue">
+          <color rgba="0 0 1 1"/>
+    </material>
+    <!-- zach -->
     <!-- LINKS -->
     <xacro:if value="${footprint_link}">

Commit message: working up to teleoperation

File: description/gazebo_control.xacro (robot description, xacro)
@@ -9,9 +9,9 @@
             <left_joint>wheel_RL_joint</left_joint>
             <right_joint>wheel_RR_joint</right_joint>
-            <wheel_separation>0.22381</wheel_separation>
-            <wheel_separation>0.22381</wheel_separation>
+            <wheel_separation>0.358</wheel_separation>
+            <wheel_separation>0.358</wheel_separation>
             <!-- dont know if its 0.057 or 0.0625 radius here took 0.057 -->
-            <wheel_diameter>0.114</wheel_diameter>
-            <wheel_diameter>0.114</wheel_diameter>
+            <wheel_diameter>0.125</wheel_diameter>
+            <wheel_diameter>0.125</wheel_diameter>
             <!-- wheel separation according to urdf 0.08214+0.14167=0.22381-->
             <!-- wheel diameter according to urdf 0.057*2 = 0.114-->

File: description/leo.urdf.xacro (robot description, xacro)
@@ -1,14 +1,14 @@
 <?xml version="1.0"?>
 <robot xmlns:xacro="http://www.ros.org/wiki/xacro" name="robot">
-      <!-- <xacro:arg name="use_ros2_control" default="true"/> -->
+      <xacro:arg name="use_ros2_control" default="true"/>
+      <xacro:arg name="sim_mode" default="false"/>
       <xacro:include filename="macros.xacro"/>
       <xacro:leo/>
-      <!-- <xacro:if value="$(arg use_ros2_control)">
-        <xacro:include filename="ros2_control.xacro" />
+      <xacro:if value="$(arg use_ros2_control)">
+            <xacro:include filename="ros2_control.xacro" />
       </xacro:if>
       <xacro:unless value="$(arg use_ros2_control)">
             <xacro:include filename="gazebo_control.xacro" />
-      </xacro:unless> -->
-      <xacro:include filename="ros2_control.xacro" />
+      </xacro:unless>
       <xacro:include filename="lidar.xacro" />
       <xacro:include filename="camera.xacro" />

File: description/ros2_control.xacro (robot description, xacro)
@@ -1,17 +1,19 @@
 <?xml version="1.0"?>
 <robot xmlns:xacro="http://www.ros.org/wiki/xacro">
-    <!-- <xacro:unless value="$(arg sim_mode)">
+    <xacro:unless value="$(arg sim_mode)">
         <ros2_control name="RealRobot" type="system">
             <hardware>
                 <plugin>diffdrive_arduino/DiffDriveArduino</plugin>
-                <param name="left_wheel_name">left_wheel_joint</param>
-                <param name="right_wheel_name">right_wheel_joint</param>
+                <param name="F_left_wheel_name">wheel_FL_joint</param>
+                <param name="F_right_wheel_name">wheel_FR_joint</param>
+                <param name="B_left_wheel_name">wheel_RL_joint</param>
+                <param name="B_right_wheel_name">wheel_RR_joint</param>
                 <param name="loop_rate">30</param>
-                <param name="device">/dev/ttyUSB0</param>
+                <param name="device">/dev/ttyACM0</param>
                 <param name="baud_rate">57600</param>
                 <param name="timeout">1000</param>
-                <param name="enc_counts_per_rev">3436</param>
+                <param name="enc_counts_per_rev">220</param>
             </hardware>
-            <joint name="left_wheel_joint">
+            <joint name="wheel_FL_joint">
                 <command_interface name="velocity">
                     <param name="min">-10</param>
@@ -21,5 +23,21 @@
                 <state_interface name="position"/>
             </joint>
-            <joint name="right_wheel_joint">
+            <joint name="wheel_FR_joint">
+                <command_interface name="velocity">
+                    <param name="min">-10</param>
+                    <param name="max">10</param>
+                </command_interface>
+                <state_interface name="velocity"/>
+                <state_interface name="position"/>
+            </joint>
+            <joint name="wheel_RL_joint">
+                <command_interface name="velocity">
+                    <param name="min">-10</param>
+                    <param name="max">10</param>
+                </command_interface>
+                <state_interface name="velocity"/>
+                <state_interface name="position"/>
+            </joint>
+            <joint name="wheel_RR_joint">
                 <command_interface name="velocity">
                     <param name="min">-10</param>
@@ -30,94 +48,48 @@
             </joint>
         </ros2_control>
-    </xacro:unless> -->
-    <!-- <xacro:if value="$(arg sim_mode)"> -->
-    <ros2_control name="RealRobot" type="system">
-        <hardware>
-            <plugin>diffdrive_arduino/DiffDriveArduino</plugin>
-            <param name="F_left_wheel_name">wheel_FL_joint</param>
-            <param name="F_right_wheel_name">wheel_FR_joint</param>
-            <param name="B_left_wheel_name">wheel_RL_joint</param>
-            <param name="B_right_wheel_name">wheel_RR_joint</param>
-            <param name="loop_rate">30</param>
-            <param name="device">/dev/ttyACM0</param>
-            <param name="baud_rate">57600</param>
-            <param name="timeout">1000</param>
-            <param name="enc_counts_per_rev">220</param>
-        </hardware>
-        <joint name="wheel_FL_joint">
-            <command_interface name="velocity">
-                <param name="min">-10</param>
-                <param name="max">10</param>
-            </command_interface>
-            <state_interface name="velocity"/>
-            <state_interface name="position"/>
-        </joint>
-        <joint name="wheel_FR_joint">
-            <command_interface name="velocity">
-                <param name="min">-10</param>
-                <param name="max">10</param>
-            </command_interface>
-            <state_interface name="velocity"/>
-            <state_interface name="position"/>
-        </joint>
-         <joint name="wheel_RL_joint">
-            <command_interface name="velocity">
-                <param name="min">-10</param>
-                <param name="max">10</param>
-            </command_interface>
-            <state_interface name="velocity"/>
-            <state_interface name="position"/>
-        </joint>
-        <joint name="wheel_RR_joint">
-            <command_interface name="velocity">
-                <param name="min">-10</param>
-                <param name="max">10</param>
-            </command_interface>
-            <state_interface name="velocity"/>
-            <state_interface name="position"/>
-        </joint>
-    </ros2_control>
-    <!-- <ros2_control name="GazeboSystem" type="system">
-        <hardware>
-            <plugin>gazebo_ros2_control/GazeboSystem</plugin>
-        </hardware>
-        <joint name="wheel_FL_joint">
-            <command_interface name="velocity">
-                <param name="min">-10</param>
-                <param name="max">10</param>
-            </command_interface>
-            <state_interface name="velocity"/>
-            <state_interface name="position"/>
-        </joint>
-        <joint name="wheel_FR_joint">
-            <command_interface name="velocity">
-                <param name="min">-10</param>
-                <param name="max">10</param>
-            </command_interface>
-            <state_interface name="velocity"/>
-            <state_interface name="position"/>
-        </joint>
-        <joint name="wheel_RL_joint">
-            <command_interface name="velocity">
-                <param name="min">-10</param>
-                <param name="max">10</param>
-            </command_interface>
-            <state_interface name="velocity"/>
-            <state_interface name="position"/>
-        </joint>
-        <joint name="wheel_RR_joint">
-            <command_interface name="velocity">
-                <param name="min">-10</param>
-                <param name="max">10</param>
-            </command_interface>
-            <state_interface name="velocity"/>
-            <state_interface name="position"/>
-        </joint>
-    </ros2_control> -->
-    <!-- </xacro:if> -->
+    </xacro:unless>
+    <xacro:if value="$(arg sim_mode)">
+        <ros2_control name="GazeboSystem" type="system">
+            <hardware>
+                <plugin>gazebo_ros2_control/GazeboSystem</plugin>
+            </hardware>
+            <joint name="wheel_FL_joint">
+                <command_interface name="velocity">
+                    <param name="min">-10</param>
+                    <param name="max">10</param>
+                </command_interface>
+                <state_interface name="velocity"/>
+                <state_interface name="position"/>
+            </joint>
+            <joint name="wheel_FR_joint">
+                <command_interface name="velocity">
+                    <param name="min">-10</param>
+                    <param name="max">10</param>
+                </command_interface>
+                <state_interface name="velocity"/>
+                <state_interface name="position"/>
+            </joint>
+            <joint name="wheel_RL_joint">
+                <command_interface name="velocity">
+                    <param name="min">-10</param>
+                    <param name="max">10</param>
+                </command_interface>
+                <state_interface name="velocity"/>
+                <state_interface name="position"/>
+            </joint>
+            <joint name="wheel_RR_joint">
+                <command_interface name="velocity">
+                    <param name="min">-10</param>
+                    <param name="max">10</param>
+                </command_interface>
+                <state_interface name="velocity"/>
+                <state_interface name="position"/>
+            </joint>
+        </ros2_control>
+    </xacro:if>
     <gazebo>
         <plugin name="gazebo_ros2_control" filename="libgazebo_ros2_control.so">
             <parameters>$(find my_bot)/config/my_controllers.yaml</parameters>
-            <!-- <parameters>$(find my_bot)/config/gaz_ros2_ctl_use_sim.yaml</parameters> -->
+            <parameters>$(find my_bot)/config/gaz_ros2_ctl_use_sim.yaml</parameters>
         </plugin>
     </gazebo>
