Commit message: adjusted some parameters

File: description/macros.xacro (robot description, xacro)
@@ -48,10 +48,23 @@
           </geometry>
         </visual>
-        <collision>
+        <!-- <collision>
           <origin xyz="0 0.04485 0" rpy="${pi/2} 0 0"/>
           <geometry>
             <cylinder radius="0.057" length="0.07"/>
           </geometry>
-        </collision>
+          <surface>
+            <friction>
+              <ode>
+                <mu>100000.0</mu>
+                <mu2>100000.0</mu2>
+              </ode>
+            </friction>
+            <contact>
+              <ode>
+                <min_depth>0.003</min_depth>
+              </ode>
+            </contact>
+          </surface>
+        </collision> -->
         <collision>
           <origin xyz="0 0.04485 0" rpy="${pi/2} 0 0"/>
@@ -59,4 +72,17 @@
             <cylinder radius="0.0625" length="0.04"/>
           </geometry>
+          <!-- <surface>
+            <friction>
+              <ode>
+                <mu>100.0</mu>
+                <mu2>100.0</mu2>
+              </ode>
+            </friction>
+            <contact>
+              <ode>
+                <min_depth>0.1</min_depth>
+              </ode>
+            </contact>
+          </surface> -->
         </collision>
         <collision>
@@ -167,6 +193,6 @@
       <child link="${link_prefix}wheel_FL_link"/>
       <axis xyz="0 -1 0"/>
-      <limit effort="2.0" velocity="6.0"/>
-      <dynamics friction="0.3125" damping="0.1"/>
+      <!-- <limit effort="2.0" velocity="6.0"/>
+      <dynamics friction="0.3125" damping="0.1"/> -->
     </joint>
     <joint name="${joint_prefix}wheel_RL_joint" type="continuous">
@@ -175,6 +201,6 @@
       <child link="${link_prefix}wheel_RL_link"/>
       <axis xyz="0 -1 0"/>
-      <limit effort="2.0" velocity="6.0"/>
-      <dynamics friction="0.3125" damping="0.1"/>
+      <!-- <limit effort="2.0" velocity="6.0"/>
+      <dynamics friction="0.3125" damping="0.1"/> -->
     </joint>
     <joint name="${joint_prefix}wheel_FR_joint" type="continuous">
@@ -183,6 +209,6 @@
       <child link="${link_prefix}wheel_FR_link"/>
       <axis xyz="0 1 0"/>
-      <limit effort="2.0" velocity="6.0"/>
-      <dynamics friction="0.3125" damping="0.1"/>
+      <!-- <limit effort="2.0" velocity="6.0"/>
+      <dynamics friction="0.3125" damping="0.1"/> -->
     </joint>
     <joint name="${joint_prefix}wheel_RR_joint" type="continuous">
@@ -191,6 +217,6 @@
       <child link="${link_prefix}wheel_RR_link"/>
       <axis xyz="0 1 0"/>
-      <limit effort="2.0" velocity="6.0"/>
-      <dynamics friction="0.3125" damping="0.1"/>
+      <!-- <limit effort="2.0" velocity="6.0"/>
+      <dynamics friction="0.3125" damping="0.1"/>  -->
     </joint>
     <xacro:if value="${default_antenna}">

Commit message: changed controller file abit, changed macros file abit - double mesh file

File: description/macros.xacro (robot description, xacro)
@@ -24,4 +24,5 @@
           <geometry>
             <mesh filename="file://$(find my_bot)/models/Rocker.dae"/>
+            <mesh filename="package://my_bot/models/Rocker.dae"/>
           </geometry>
         </visual>
@@ -29,4 +30,5 @@
           <geometry>
             <mesh filename="file://$(find my_bot)/models/Rocker_outline.stl"/>
+            <mesh filename="package://my_bot/models/Rocker_outline.stl"/>
           </geometry>
         </collision>
@@ -46,47 +48,17 @@
           <geometry>
             <mesh filename="file://$(find my_bot)/models/Wheel${model}.dae"/>
+            <mesh filename="package://my_bot/models/Wheel${model}.dae"/>
           </geometry>
         </visual>
-        <!-- <collision>
+        <collision>
           <origin xyz="0 0.04485 0" rpy="${pi/2} 0 0"/>
           <geometry>
-            <cylinder radius="0.057" length="0.07"/>
-          </geometry>
-          <surface>
-            <friction>
-              <ode>
-                <mu>100000.0</mu>
-                <mu2>100000.0</mu2>
-              </ode>
-            </friction>
-            <contact>
-              <ode>
-                <min_depth>0.003</min_depth>
-              </ode>
-            </contact>
-          </surface>
-        </collision> -->
-        <collision>
-          <origin xyz="0 0.04485 0" rpy="${pi/2} 0 0"/>
-          <geometry>
             <cylinder radius="0.0625" length="0.04"/>
           </geometry>
-          <!-- <surface>
-            <friction>
-              <ode>
-                <mu>100.0</mu>
-                <mu2>100.0</mu2>
-              </ode>
-            </friction>
-            <contact>
-              <ode>
-                <min_depth>0.1</min_depth>
-              </ode>
-            </contact>
-          </surface> -->
         </collision>
         <collision>
           <geometry>
             <mesh filename="file://$(find my_bot)/models/Wheel_outline.stl"/>
+            <mesh filename="package://my_bot/models/Wheel_outline.stl"/>
           </geometry>
         </collision>
@@ -117,4 +89,5 @@
         <geometry>
           <mesh filename="file://$(find my_bot)/models/Chassis.dae"/>
+          <mesh filename="package://my_bot/models/Chassis.dae"/>
         </geometry>
       </visual>
@@ -122,4 +95,5 @@
         <geometry>
           <mesh filename="file://$(find my_bot)/models/Chassis_outline.stl"/>
+          <mesh filename="package://my_bot/models/Chassis_outline.stl"/>
         </geometry>
       </collision>
@@ -144,4 +118,5 @@
           <geometry>
             <mesh filename="file://$(find my_bot)/models/Antenna.dae"/>
+            <mesh filename="package://my_bot/models/Antenna.dae"/>
           </geometry>
         </visual>
@@ -242,4 +217,37 @@
       <child link="${link_prefix}imu_frame"/>
     </joint> -->
+    <!-- wheel ODE properties -->
+    <!-- <gazebo reference="${link_prefix}wheel_FL_link">
+      <kp>1e6</kp>
+      <kd>100.0</kd>
+      <mu1>3.0</mu1>
+      <mu2>1.0</mu2>
+      <fdir1>1 0 0</fdir1>
+      <minDepth>0.003</minDepth>
+    </gazebo>
+    <gazebo reference="${link_prefix}wheel_FR_link">
+      <kp>1e6</kp>
+      <kd>100.0</kd>
+      <mu1>3.0</mu1>
+      <mu2>1.0</mu2>
+      <fdir1>1 0 0</fdir1>
+      <minDepth>0.003</minDepth>
+    </gazebo>
+    <gazebo reference="${link_prefix}wheel_RL_link">
+      <kp>1e6</kp>
+      <kd>100.0</kd>
+      <mu1>3.0</mu1>
+      <mu2>1.0</mu2>
+      <fdir1>1 0 0</fdir1>
+      <minDepth>0.003</minDepth>
+    </gazebo>
+    <gazebo reference="${link_prefix}wheel_RR_link">
+      <kp>1e6</kp>
+      <kd>100.0</kd>
+      <mu1>3.0</mu1>
+      <mu2>1.0</mu2>
+      <fdir1>1 0 0</fdir1>
+      <minDepth>0.003</minDepth>
+    </gazebo> -->
   </xacro:macro>
 </robot>

Commit message: fixed robot model not being able to load in rviz2 dev machine when running launch on jetson

File: description/macros.xacro (robot description, xacro)
@@ -23,12 +23,20 @@
         <visual>
           <geometry>
-            <mesh filename="file://$(find my_bot)/models/Rocker.dae"/>
-            <mesh filename="package://my_bot/models/Rocker.dae"/>
+            <xacro:if value="$(arg sim_mode)">
+              <mesh filename="file://$(find my_bot)/models/Rocker.dae"/>
+            </xacro:if>
+            <xacro:unless value="$(arg sim_mode)">
+              <mesh filename="package://my_bot/models/Rocker.dae"/>
+            </xacro:unless>
           </geometry>
         </visual>
         <collision>
           <geometry>
-            <mesh filename="file://$(find my_bot)/models/Rocker_outline.stl"/>
-            <mesh filename="package://my_bot/models/Rocker_outline.stl"/>
+            <xacro:if value="$(arg sim_mode)">
+              <mesh filename="file://$(find my_bot)/models/Rocker_outline.stl"/>
+            </xacro:if>
+            <xacro:unless value="$(arg sim_mode)">
+              <mesh filename="package://my_bot/models/Rocker_outline.stl"/>
+            </xacro:unless>
           </geometry>
         </collision>
@@ -47,6 +55,10 @@
         <visual>
           <geometry>
-            <mesh filename="file://$(find my_bot)/models/Wheel${model}.dae"/>
-            <mesh filename="package://my_bot/models/Wheel${model}.dae"/>
+            <xacro:if value="$(arg sim_mode)">
+              <mesh filename="file://$(find my_bot)/models/Wheel${model}.dae"/>
+            </xacro:if>
+            <xacro:unless value="$(arg sim_mode)">
+              <mesh filename="package://my_bot/models/Wheel${model}.dae"/>
+            </xacro:unless>
           </geometry>
         </visual>
@@ -59,6 +71,10 @@
         <collision>
           <geometry>
-            <mesh filename="file://$(find my_bot)/models/Wheel_outline.stl"/>
-            <mesh filename="package://my_bot/models/Wheel_outline.stl"/>
+            <xacro:if value="$(arg sim_mode)">
+              <mesh filename="file://$(find my_bot)/models/Wheel_outline.stl"/>
+            </xacro:if>
+            <xacro:unless value="$(arg sim_mode)">
+              <mesh filename="package://my_bot/models/Wheel_outline.stl"/>
+            </xacro:unless>
           </geometry>
         </collision>
@@ -88,12 +104,20 @@
       <visual>
         <geometry>
-          <mesh filename="file://$(find my_bot)/models/Chassis.dae"/>
-          <mesh filename="package://my_bot/models/Chassis.dae"/>
+          <xacro:if value="$(arg sim_mode)">
+            <mesh filename="file://$(find my_bot)/models/Chassis.dae"/>
+          </xacro:if>
+          <xacro:unless value="$(arg sim_mode)">
+            <mesh filename="package://my_bot/models/Chassis.dae"/>
+          </xacro:unless>
         </geometry>
       </visual>
       <collision>
         <geometry>
-          <mesh filename="file://$(find my_bot)/models/Chassis_outline.stl"/>
-          <mesh filename="package://my_bot/models/Chassis_outline.stl"/>
+          <xacro:if value="$(arg sim_mode)">
+            <mesh filename="file://$(find my_bot)/models/Chassis_outline.stl"/>
+          </xacro:if>
+          <xacro:unless value="$(arg sim_mode)">
+            <mesh filename="package://my_bot/models/Chassis_outline.stl"/>
+          </xacro:unless>
         </geometry>
       </collision>
@@ -117,6 +141,10 @@
         <visual>
           <geometry>
-            <mesh filename="file://$(find my_bot)/models/Antenna.dae"/>
-            <mesh filename="package://my_bot/models/Antenna.dae"/>
+            <xacro:if value="$(arg sim_mode)">
+              <mesh filename="file://$(find my_bot)/models/Antenna.dae"/>
+            </xacro:if>
+            <xacro:unless value="$(arg sim_mode)">
+              <mesh filename="package://my_bot/models/Antenna.dae"/>
+            </xacro:unless>
           </geometry>
         </visual>
